Commit message: added joints and collisions

File: urdf/dd_robot.urdf (robot description, URDF)
Before this commit: robot dd_robot, 1 links, 0 joints
Links:
- added link left_wheel; visual cylinder length=0.1 radius=0.2
- added link right_wheel; visual cylinder length=0.1 radius=0.2
- link base_link: geometry visual box size=0.5 0.5 0.25; visual sphere radius=0.05
Joints:
- added joint joint_left_wheel: type continuous, parent base_link, child left_wheel, origin xyz=0 0.30 0 rpy=0 0 0, axis 0 1 0
- added joint joint_right_wheel: type continuous, parent base_link, child right_wheel, origin xyz=0 -0.30 0 rpy=0 0 0, axis 0 1 0

Commit message: added inertia to the links

File: urdf/dd_robot.urdf (robot description, URDF)
Before this commit: robot dd_robot, 3 links, 2 joints
Links:
- link base_link: mass None -> 5; geometry collision box size=0.5 0.5 0.25; collision sphere radius=0.05
- link left_wheel: mass None -> 0.5; geometry collision cylinder length=0.1 radius=0.2; visual cylinder length=0.1 radius=0.2
- link right_wheel: mass None -> 0.5; geometry collision cylinder length=0.1 radius=0.2; visual cylinder length=0.1 radius=0.2
